Commit message: feat(simulation): put a camera on the simulated Mini
Adds a stereo-left camera at the real capture format — 480x270, 30 Hz,
matching what the vehicle publishes so the perception code cannot tell
the difference — and the Sensors system the world needs to render it
at all. Elixir now receives simulated frames at 28.7 Hz.

**Compressed, not raw, and the difference is not cosmetic.** A
480x270 rgb8 frame is 389 KB; at 30 Hz that is 11.6 MB/s. Putting it
on the Zenoh fabric does not work: a subscriber that cannot drain it
that fast received **one frame every fifteen seconds**, because zenoh
drops what the link will not carry. The failure looks like a broken
topic rather than a saturated one. Cameras therefore go through
`ros_gz_image image_bridge`, whose image_transport JPEG variant is
about 6.5 KB — roughly what the real vehicle publishes — and raw
pixels stay inside gz-transport where they are cheap. Raw on the wire
looked preferable on the grounds that a simulated camera has no reason
to invent a JPEG; measurement disagreed.

Two Gazebo traps, both silent:

  * A **massless link is dropped** in URDF-to-SDF conversion and its
    <gazebo> elements are reparented — here all the way up to
    base_link, which puts the camera somewhere else entirely while
    still rendering happily. The sensor hangs off the mount, which has
    mass, and only the reported frame_id names the optical child.
  * Without the **Sensors system** in the world a camera loads,
    reports no error and publishes nothing.

Headless rendering needs no GPU: ogre2 falls back to software
rasterisation and still holds 28.2 Hz at RTF 0.93.

`Image.parse/1` completes the codec so the bridge can consume images
as well as emit them. It has to undo the same two irregularities the
encoder introduces — the unpadded `encoding` string and the
realignment after `is_bigendian` — and the second depends on the
offset from the body origin, so it parses against the whole body
rather than the remainder.

Frames arrive stamped `stereo_left_optical`, decoded as
"rgb8; jpeg compressed bgr8".

File: vehicles/ovcs_mini/description/ovcs_mini.urdf.xacro (robot description, xacro)
@@ -35,4 +35,5 @@
   <xacro:include filename="../../common/materials.xacro" />
   <xacro:include filename="wheels.xacro" />
+  <xacro:include filename="sensors.xacro" />
   <!-- ── Measured: Traxxas Slash 4x4 specification ──────────────── -->
   <xacro:property name="wheelbase"     value="0.324" />
@@ -132,4 +133,20 @@
   <xacro:steered_wheel name="front_right" side="-1"
                        x="${half_wheelbase}" />
+  <!-- ── Sensors ────────────────────────────────────────────────── -->
+  <!-- Matches the real vehicle's capture: 480x270 at 30 Hz. The
+       resolution is not arbitrary — it is what the stereo pipeline was
+       tuned to, trading depth precision at range for a 0.55 m near
+       clip and half the SGBM cost. Simulating something else would
+       measure a pipeline the vehicle does not run.
+       The stereo pair straddles the vehicle centreline at the
+       measured 90 mm baseline. Height and forward offset are the
+       simulation's own choice, since the real ones were never
+       measured — see sensors.xacro. -->
+  <xacro:property name="baseline" value="0.090" />
+  <xacro:property name="camera_x" value="0.10" />
+  <xacro:property name="camera_z" value="0.12" />
+  <xacro:sim_camera name="stereo_left"  x="${camera_x}" y="${baseline / 2}"
+                    z="${camera_z}" topic="stereo/left/image_raw"
+                    width="480" height="270" fov_deg="70" rate="30" />
   <xacro:include filename="gazebo_ackermann.xacro" />
 </robot>

Commit message: fix(ovcs_mini): put the cameras where they actually are
Measured off the vehicle, replacing two numbers that were guessed and
one that was invented.

**Forward offset was 58 mm out.** `base_link` sits midway between the
axles, so with a 324 mm wheelbase the front axle is 162 mm ahead of
it. The camera bar is 120 mm behind that axle, putting the lenses at
42 mm forward of base_link — not the 100 mm the placeholder claimed.
Every detection the vehicle published was correctly positioned
relative to the camera and 58 mm too far forward relative to the car.

**Field of view was invented.** The simulated cameras had a
plausible-looking 70 degrees. The vehicle's own calibration says
otherwise: the rectified P gives fx = 779.55 at 640 wide, which is
584.66 at the 480 the pipeline captures — about 45 degrees.

That distinction is not cosmetic, because focal length is what the
stereo maths runs on. With the real value f*B comes out at 52.6 and
the near clip at 52.6 / 96 = 0.55 m, exactly the figure the vehicle
was tuned to; at 70 degrees it would have been 0.32, and the simulator
would have quietly modelled a camera that sees closer than the real
one. The FOV is now derived from the measured focal length rather than
stated, so the two cannot drift apart.

**Baseline confirmed at 90 mm** — that one was right.

Adds the right camera, so the simulator now has a stereo pair rather
than a single eye. Verified through the bridge over Zenoh: both sides
at 27.9 Hz with all 279 timestamps shared, which is what the backend's
pair matching needs, and the published camera_info gives -tx/fx =
0.09 m.

The bar also carries an FPV camera between the two. Deliberately not
modelled: nothing in the perception path reads it.

z is still the original guess — the last unmeasured number in the
vehicle's geometry, marked TODO in both places.

File: vehicles/ovcs_mini/description/ovcs_mini.urdf.xacro (robot description, xacro)
@@ -139,14 +139,34 @@
        clip and half the SGBM cost. Simulating something else would
        measure a pipeline the vehicle does not run.
-       The stereo pair straddles the vehicle centreline at the
-       measured 90 mm baseline. Height and forward offset are the
-       simulation's own choice, since the real ones were never
-       measured — see sensors.xacro. -->
+       Measured off the vehicle:
+         baseline  90 mm, straddling the centreline
+         position  120 mm behind the front axle
+       The front axle is half a wheelbase ahead of base_link, so the
+       bar sits at 162 - 120 = 42 mm forward of it — not the 100 mm
+       that was guessed, which put the cameras 58 mm too far forward
+       and biased every detection by that much.
+       The bar also carries a third, FPV camera between the two. It is
+       not modelled: nothing in the perception path reads it. -->
   <xacro:property name="baseline" value="0.090" />
-  <xacro:property name="camera_x" value="0.10" />
+  <!-- From the vehicle's own calibration
+       (vehicles/ovcs_mini/priv/calibration/stereo_left.yaml): the
+       rectified P gives fx = 779.55 at 640 wide, and the pipeline
+       captures at 480, so fx scales to 779.55 * 0.75 = 584.66.
+       That is a ~45 degree horizontal field of view, not the ~70 a
+       wide-angle module would suggest, and it is what makes the
+       simulated depth behave like the real one: f*B = 52.6, so the
+       near clip lands at 52.6 / 96 = 0.55 m — the figure the vehicle
+       was tuned to. -->
+  <xacro:property name="focal_px" value="${779.54677 * 480 / 640}" />
+  <xacro:property name="camera_x" value="${half_wheelbase - 0.120}" />
+  <!-- TODO: still unmeasured. Lens centre height above the ground. -->
   <xacro:property name="camera_z" value="0.12" />
+  <!-- Left is +y in REP-103. -->
   <xacro:sim_camera name="stereo_left"  x="${camera_x}" y="${baseline / 2}"
                     z="${camera_z}" topic="stereo/left/image_raw"
-                    width="480" height="270" fov_deg="70" rate="30" />
+                    width="480" height="270" focal_px="${focal_px}" rate="30" />
+  <xacro:sim_camera name="stereo_right" x="${camera_x}" y="${-baseline / 2}"
+                    z="${camera_z}" topic="stereo/right/image_raw"
+                    width="480" height="270" focal_px="${focal_px}" rate="30" />
   <xacro:include filename="gazebo_ackermann.xacro" />
 </robot>

File: vehicles/ovcs_mini/description/sensors.xacro (robot description, xacro)
@@ -29,5 +29,5 @@
     code should not be able to tell the difference.
   -->
-  <xacro:macro name="sim_camera" params="name x y z topic width height fov_deg rate">
+  <xacro:macro name="sim_camera" params="name x y z topic width height focal_px rate">
     <link name="${name}_link">
       <visual>
@@ -78,5 +78,12 @@
         <frame_id>${name}_optical</frame_id>
         <camera>
-          <horizontal_fov>${fov_deg * pi / 180.0}</horizontal_fov>
+          <!-- Field of view is derived from the *measured* focal
+               length rather than chosen, because it is focal length
+               that the stereo pipeline actually depends on: the near
+               clip is f*B / num_disparities and depth error goes as
+               Z^2 / (f*B). A simulator with a plausible-looking FOV
+               but the wrong f models a different camera and quietly
+               reports different depth behaviour than the vehicle. -->
+          <horizontal_fov>${2 * atan2(width / 2.0, focal_px)}</horizontal_fov>
           <image>
             <width>${width}</width>

Commit message: feat(ros_bridge): a simulated BNO085, consumed like the real one
The simulator had no IMU: the model declared none, the worlds did not
load the IMU system, and against Gazebo the host bridge published
/imu from the Dummy driver's static fixtures — plausible-looking
constants on a dashboard.

The model now carries an IMU sensor at the BNO085's (still
unmeasured, like the cameras') mounting point, publishing on
`imu_raw` at the chip's 100 Hz. `RosBridge.Imu.Zenoh` consumes that
topic and casts the same `{:imu_sample, %Sample{}}` messages the
hardware driver does, so `Publishers.Imu` republishes on `/imu`
unchanged — only the driver differs between the car and the simulated
car, the same pattern as the cameras. Two topic names on purpose: one
name for both would have the bridge republishing onto the topic it is
consuming.

One message fans out into the three sample kinds the hardware
produces; `sensor_msgs/Imu` is already SI, so it is a fan-out, not a
conversion. No <noise> on the sensor yet: a perfect heading is fine
while Gazebo also owns the odometry, and the day the bridge's dead
reckoning runs against the simulator, noise measured from the real
chip belongs there.

The IMU has its own Gazebo system, separate from Sensors; without it
a declared sensor publishes nothing, silently. Both worlds load it.

Assisted-by: Claude:claude-fable-5

File: vehicles/ovcs_mini/description/ovcs_mini.urdf.xacro (robot description, xacro)
@@ -169,4 +169,8 @@
                     z="${camera_z}" topic="stereo/right/image_raw"
                     width="480" height="270" focal_px="${focal_px}" rate="30" />
+  <!-- TODO: placeholder, like the camera transform — the BNO085's
+       real mounting position has not been measured. Harmless while
+       only orientation is consumed. 100 Hz is the BNO085's cadence. -->
+  <xacro:sim_imu name="imu" x="0" y="0" z="0.05" rate="100" />
   <xacro:include filename="gazebo_ackermann.xacro" />
 </robot>

File: vehicles/ovcs_mini/description/sensors.xacro (robot description, xacro)
@@ -102,3 +102,40 @@
     </gazebo>
   </xacro:macro>
+  <!--
+    The simulated BNO085. One link with just enough mass to survive
+    the URDF-to-SDF conversion (massless links are dropped and their
+    <gazebo> elements silently reparented — see the camera comment
+    above), and a stock Gazebo IMU sensor on it. The world must load
+    `gz-sim-imu-system`; a sensor without its system publishes
+    nothing, silently.
+    The topic is `imu_raw`, not `imu`, on purpose: the bridge's
+    `RosBridge.Imu.Zenoh` driver consumes this and `Publishers.Imu`
+    republishes on `/imu`, exactly as on the vehicle. One name for
+    both would have the bridge republishing onto the topic it reads.
+    No <noise> yet: a perfect heading. Fine while Gazebo also owns
+    the odometry; the day the bridge's dead reckoning runs against
+    the simulator, noise and bias measured from the real BNO085
+    belong here, because a drift-free heading would make that loop
+    prove less than it appears to.
+  -->
+  <xacro:macro name="sim_imu" params="name x y z rate">
+    <link name="${name}_link">
+      <xacro:inertial_box mass="0.005" x="0.014" y="0.012" z="0.002">
+        <origin xyz="0 0 0" rpy="0 0 0" />
+      </xacro:inertial_box>
+    </link>
+    <joint name="${name}_joint" type="fixed">
+      <parent link="base_link" />
+      <child link="${name}_link" />
+      <origin xyz="${x} ${y} ${z}" rpy="0 0 0" />
+    </joint>
+    <gazebo reference="${name}_link">
+      <sensor name="${name}" type="imu">
+        <always_on>1</always_on>
+        <update_rate>${rate}</update_rate>
+        <topic>imu_raw</topic>
+        <frame_id>${name}_link</frame_id>
+      </sensor>
+    </gazebo>
+  </xacro:macro>
 </robot>

Commit message: Use the OVCS Mini's rolling wheel radius
A 3.00 m drive read 3.15 m with the physical 0.0548 m; under load the
tyres roll on 0.0522 m, and the same drive then reads 2.965 m.

Assisted-by: Claude:claude-opus-5-5

File: vehicles/ovcs_mini/description/ovcs_mini.urdf.xacro (robot description, xacro)
@@ -37,5 +37,5 @@
   <xacro:property name="wheelbase"     value="0.324" />
   <xacro:property name="track"         value="0.296" />
-  <xacro:property name="wheel_radius"  value="0.0548" />
+  <xacro:property name="wheel_radius"  value="0.0522" />
   <xacro:property name="body_length"   value="0.568" />
   <xacro:property name="body_width"    value="0.296" />

Commit message: Set the OVCS Mini stereo camera height to the measured 185 mm
Assisted-by: Claude:claude-opus-5-5

File: vehicles/ovcs_mini/description/ovcs_mini.urdf.xacro (robot description, xacro)
@@ -81,9 +81,9 @@
   <!-- Gazebo 10 velocity mode uses L / sin(parameter), not L / tan(parameter). -->
   <xacro:property name="gazebo_steering_limit" value="${asin(tan(steering_limit))}" />
-  <!-- Stereo geometry; camera height remains an estimate. -->
+  <!-- Stereo geometry. -->
   <xacro:property name="baseline" value="0.090" />
   <xacro:property name="focal_px" value="${779.54677 * 480 / 640}" />
   <xacro:property name="camera_x" value="${half_wheelbase - 0.120}" />
-  <xacro:property name="camera_z" value="0.12" />
+  <xacro:property name="camera_z" value="0.185" />
   <!-- ── base_link ──────────────────────────────────────────────── -->
   <!-- Deliberately empty. A link with no inertia is the conventional

File: vehicles/ovcs_mini/description/sensors.xacro (robot description, xacro)
@@ -2,6 +2,6 @@
 <!--
   Simulated sensors.
-  Sensor offsets are model parameters; the camera height and IMU mount
-  remain estimates. Exact placement in simulation does not validate the
+  Sensor offsets are model parameters; the IMU mount remains an
+  estimate. Exact placement in simulation does not validate the
   placement of the physical sensor.
   ## Frames

Commit message: Correct vehicle geometry and sensor freshness for navigation
Reference Ackermann odometry at the rear axle and include the base_link
lever arm in its published pose and twist. Require fresh wheel and IMU
samples, and reject delayed or replayed stamped velocity commands.

Feed depth and point clouds from the same disparity data, tighten stereo
pairing and place the left camera at its offset from the centreline.

Assisted-by: Codex:gpt-6

File: vehicles/ovcs_mini/description/ovcs_mini.urdf.xacro (robot description, xacro)
@@ -91,4 +91,10 @@
        double-count the chassis. -->
   <link name="base_link" />
+  <link name="rear_axle" />
+  <joint name="rear_axle_joint" type="fixed">
+    <parent link="base_link" />
+    <child link="rear_axle" />
+    <origin xyz="${-half_wheelbase} 0 0" rpy="0 0 0" />
+  </joint>
   <!-- ── Chassis ────────────────────────────────────────────────── -->
   <joint name="chassis_joint" type="fixed">

Commit message: Recalibrate the OVCS Mini stereo cameras
The mount moved: with the previous calibration the rectified rows were
28 px apart and most of the image found no match. The new calibration,
solved at the 480x270 capture size, puts them within 0.5 px, and a
fleece target at a measured 2.30 m reads 2.17-2.23 m, so the right
camera's cx correction for a constant disparity offset is no longer
needed. f*B is 55.6, which moves the near clip to 0.58 m; the
simulated camera and the figures derived from it follow.

camera_calibration 7.1.7 predates Lyrical's rclpy and NumPy 2:
cameracalibrator crashed at start and on SAVE, and buffered output
hid CALIBRATE's results.

Assisted-by: Claude:claude-opus-5-5

File: vehicles/ovcs_mini/description/ovcs_mini.urdf.xacro (robot description, xacro)
@@ -83,5 +83,5 @@
   <!-- Stereo geometry. -->
   <xacro:property name="baseline" value="0.090" />
-  <xacro:property name="focal_px" value="${779.54677 * 480 / 640}" />
+  <xacro:property name="focal_px" value="617.02" />
   <xacro:property name="camera_x" value="${half_wheelbase - 0.120}" />
   <xacro:property name="camera_z" value="0.185" />
@@ -124,5 +124,5 @@
   <!-- Matches the real vehicle's capture: 480x270 at 30 Hz. The
        resolution is not arbitrary — it is what the stereo pipeline was
-       tuned to, trading depth precision at range for a 0.55 m near
+       tuned to, trading depth precision at range for a 0.58 m near
        clip and half the SGBM cost. Simulating something else would
        measure a pipeline the vehicle does not run.
@@ -138,11 +138,9 @@
   <!-- From the vehicle's own calibration
        (vehicles/ovcs_mini/priv/calibration/stereo_left.yaml): the
-       rectified P gives fx = 779.55 at 640 wide, and the pipeline
-       captures at 480, so fx scales to 779.55 * 0.75 = 584.66.
-       That is a ~45 degree horizontal field of view, not the ~70 a
+       rectified P gives fx = 617.02 at the 480 px capture width.
+       That is a ~43 degree horizontal field of view, not the ~70 a
        wide-angle module would suggest, and it is what makes the
-       simulated depth behave like the real one: f*B = 52.6, so the
-       near clip lands at 52.6 / 96 = 0.55 m — the figure the vehicle
-       was tuned to. -->
+       simulated depth behave like the real one: f*B = 55.5, so the
+       near clip lands at 55.5 / 96 = 0.58 m. -->
   <!-- TODO: still unmeasured. Lens centre height above the ground. -->
   <!-- Left is +y in REP-103. -->

File: vehicles/ovcs_mini/description/sensors.xacro (robot description, xacro)
@@ -88,5 +88,5 @@
           </image>
           <clip>
-            <!-- Near plane well inside the stereo near clip (0.55 m on
+            <!-- Near plane well inside the stereo near clip (0.58 m on
                  the real rig) so the simulation is not the thing that
                  limits close range. -->

Commit message: Use the whole sensor on the OVCS Mini's stereo cameras
libcamera's own pick for the 480x270 output is a centre crop of the
IMX708, 42.5° of horizontal field of view. The 2304x1296 mode bins the
whole sensor: 65° after rectification, and f*B falls from 55.6 to 34.5,
which brings the near clip from 0.58 to 0.36 m for 5.8 cm of depth
precision at 2 m instead of 3.6. The calibration is solved for that
mode (0.64 px RMS, rows within 0.4 px), and the simulated camera and
its calibration follow; the simulator's calibration had kept the
focal length from before the previous recalibration.

Assisted-by: Claude:claude-opus-5-5

File: vehicles/ovcs_mini/description/ovcs_mini.urdf.xacro (robot description, xacro)
@@ -83,5 +83,5 @@
   <!-- Stereo geometry. -->
   <xacro:property name="baseline" value="0.090" />
-  <xacro:property name="focal_px" value="617.02" />
+  <xacro:property name="focal_px" value="379.03" />
   <xacro:property name="camera_x" value="${half_wheelbase - 0.120}" />
   <xacro:property name="camera_z" value="0.185" />
@@ -124,5 +124,5 @@
   <!-- Matches the real vehicle's capture: 480x270 at 30 Hz. The
        resolution is not arbitrary — it is what the stereo pipeline was
-       tuned to, trading depth precision at range for a 0.58 m near
+       tuned to, trading depth precision at range for a 0.36 m near
        clip and half the SGBM cost. Simulating something else would
        measure a pipeline the vehicle does not run.
@@ -138,9 +138,10 @@
   <!-- From the vehicle's own calibration
        (vehicles/ovcs_mini/priv/calibration/stereo_left.yaml): the
-       rectified P gives fx = 617.02 at the 480 px capture width.
-       That is a ~43 degree horizontal field of view, not the ~70 a
-       wide-angle module would suggest, and it is what makes the
-       simulated depth behave like the real one: f*B = 55.5, so the
-       near clip lands at 55.5 / 96 = 0.58 m. -->
+       rectified P gives fx = 379.03 at the 480 px capture width, with
+       the cameras binning the whole sensor.
+       That is a ~65 degree horizontal field of view after
+       rectification, and it is what makes the simulated depth behave
+       like the real one: f*B = 34.1, so the near clip lands at
+       34.1 / 96 = 0.36 m. -->
   <!-- TODO: still unmeasured. Lens centre height above the ground. -->
   <!-- Left is +y in REP-103. -->

File: vehicles/ovcs_mini/description/sensors.xacro (robot description, xacro)
@@ -88,5 +88,5 @@
           </image>
           <clip>
-            <!-- Near plane well inside the stereo near clip (0.58 m on
+            <!-- Near plane well inside the stereo near clip (0.36 m on
                  the real rig) so the simulation is not the thing that
                  limits close range. -->
