Commit message: Simulate the OVCS Mini's lidar and rear ultrasonics
Gazebo gpu_lidar sensors stand in for the RPLIDAR and, as 60° fans,
for the two A02YYUW. RosBridge.Lidar.Zenoh and
RosBridge.Rangefinder.Zenoh turn their LaserScans into the samples the
hardware drivers produce, so the bridge publishes /scan and
ultrasound/rear_* as on the vehicle. The LaserScan and Range
publishers stamp through Timing, on simulator time when a /clock is
followed.

Assisted-by: Claude:claude-opus-5-5

File: vehicles/ovcs_mini/description/ovcs_mini.urdf.xacro (robot description, xacro)
@@ -65,4 +65,5 @@
   <xacro:property name="camera_mass" value="0.005" />
   <xacro:property name="imu_mass" value="0.005" />
+  <xacro:property name="ray_sensor_mass" value="0.005" />
   <!-- ── Derived ────────────────────────────────────────────────── -->
   <xacro:property name="half_wheelbase" value="${wheelbase / 2}" />
@@ -156,4 +157,16 @@
        only orientation is consumed. 100 Hz is the BNO085's cadence. -->
   <xacro:sim_imu name="imu" x="0" y="0" z="0.05" rate="100" />
+  <!-- Mounts as the ROS bridge's static transforms have them
+       (`OvcsMini`'s `lidar_transform/0`, `rear_ultrasound_transforms/0`).
+       The lidar's row stops a step short of +π, which would repeat its first ray. -->
+  <xacro:sim_ray name="lidar" x="-0.137" y="0" z="0.205" yaw="0"
+                 topic="scan_raw" samples="500"
+                 min_angle="${-pi}" max_angle="${pi - 2 * pi / 500}" min_range="0.05" max_range="12.0" rate="10" />
+  <xacro:sim_ray name="ultrasound_rear_left" x="-0.2976" y="0.0418" z="0.110"
+                 yaw="${radians(170)}" topic="ultrasound/rear_left_raw" samples="13"
+                 min_angle="${radians(-30)}" max_angle="${radians(30)}" min_range="0.03" max_range="4.5" rate="10" />
+  <xacro:sim_ray name="ultrasound_rear_right" x="-0.2976" y="-0.0418" z="0.110"
+                 yaw="${radians(-170)}" topic="ultrasound/rear_right_raw" samples="13"
+                 min_angle="${radians(-30)}" max_angle="${radians(30)}" min_range="0.03" max_range="4.5" rate="10" />
   <xacro:include filename="gazebo_ackermann.xacro" />
 </robot>

File: vehicles/ovcs_mini/description/sensors.xacro (robot description, xacro)
@@ -135,3 +135,44 @@
     </gazebo>
   </xacro:macro>
+  <!--
+    A planar `gpu_lidar`: `samples` rays from `min_angle` to `max_angle`,
+    both included, published as a LaserScan on `topic`. It stands in for
+    the RPLIDAR and, as a horizontal fan that keeps the floor out of the
+    beam, for each A02YYUW; `RosBridge.Lidar.Zenoh` and
+    `RosBridge.Rangefinder.Zenoh` consume them.
+  -->
+  <xacro:macro name="sim_ray" params="name x y z yaw topic samples min_angle max_angle min_range max_range rate">
+    <link name="${name}_link">
+      <xacro:inertial_box mass="${ray_sensor_mass}" x="0.02" y="0.02" z="0.02">
+        <origin xyz="0 0 0" rpy="0 0 0" />
+      </xacro:inertial_box>
+    </link>
+    <joint name="${name}_joint" type="fixed">
+      <parent link="base_link" />
+      <child link="${name}_link" />
+      <origin xyz="${x} ${y} ${z}" rpy="0 0 ${yaw}" />
+    </joint>
+    <gazebo reference="${name}_link">
+      <sensor name="${name}" type="gpu_lidar">
+        <always_on>1</always_on>
+        <update_rate>${rate}</update_rate>
+        <visualize>false</visualize>
+        <topic>${topic}</topic>
+        <frame_id>${name}_link</frame_id>
+        <lidar>
+          <scan>
+            <horizontal>
+              <samples>${samples}</samples>
+              <min_angle>${min_angle}</min_angle>
+              <max_angle>${max_angle}</max_angle>
+            </horizontal>
+          </scan>
+          <range>
+            <min>${min_range}</min>
+            <max>${max_range}</max>
+          </range>
+        </lidar>
+      </sensor>
+    </gazebo>
+  </xacro:macro>
 </robot>

Commit message: Measure the simulator plant's speed at the wheels
The vehicle's motor and shaft sensors measure the wheels, not the body,
so the plant now takes the wheel joints' mean velocity on /joint_states
times the wheel radius instead of the body speed on /simulator/odom,
which is left for comparison with /odom. A wheel spinning in place
reads as moving, as it would on the vehicle. Nothing parses
nav_msgs/Odometry any more, so its decoder goes.

AckermannSteering drives the wheels at the commanded velocity, so the
OVCS Mini's wheel joints get an effort limit, the torque its motor's
current gives each wheel: against a box, the wheels stall and /odom
stops 1.8 cm short of the model, where without it /odom ran on 1.64 m.
A steady 0.6 rad/s arc turns at 0.5787 rad/s, against 0.5835 without
the limit.

Assisted-by: Claude:claude-opus-5-5

File: vehicles/ovcs_mini/description/ovcs_mini.urdf.xacro (robot description, xacro)
@@ -66,4 +66,8 @@
   <xacro:property name="imu_mass" value="0.005" />
   <xacro:property name="ray_sensor_mass" value="0.005" />
+  <!-- The drive force the simulator plant gives the VESC's 10 A at its
+       0.5 m/s² per ampere (`OvcsMini`), shared by the four wheels: a
+       wheel held back stalls instead of spinning at the commanded speed. -->
+  <xacro:property name="wheel_max_torque" value="${total_mass * 0.5 * 10 * wheel_radius / 4}" />
   <!-- ── Derived ────────────────────────────────────────────────── -->
   <xacro:property name="half_wheelbase" value="${wheelbase / 2}" />

File: vehicles/ovcs_mini/description/wheels.xacro (robot description, xacro)
@@ -47,4 +47,6 @@
               rpy="${-pi/2} 0 0" />
       <axis xyz="0 0 1" />
+      <!-- URDF requires a velocity with the effort; the drive's own limit applies. -->
+      <limit effort="${wheel_max_torque}" velocity="1000" />
       <dynamics damping="0.01" friction="0.0" />
     </joint>
@@ -87,4 +89,6 @@
       <origin xyz="0 0 0" rpy="${-pi/2} 0 0" />
       <axis xyz="0 0 1" />
+      <!-- URDF requires a velocity with the effort; the drive's own limit applies. -->
+      <limit effort="${wheel_max_torque}" velocity="1000" />
       <dynamics damping="0.01" friction="0.0" />
     </joint>
