Commit message: Check the OVCS Mini model against its Elixir side, and trim the stack
- geometry_test.exs checks the sensor mounts against the bridge's
  static transforms, and the wheel torque's motor current and
  acceleration per ampere, now named xacro properties, against the
  composer and the simulated hardware. The chassis mass leaves out the
  three ray sensors' links.
- AckermannSteering's odometry tags go: nothing bridges that odometry.
  Comments describing removed behaviour or another model's history are
  cut, the wheel radius matches geometry/0, and the world names its
  stereo figures as the OVCS Mini's.
- The Gazebo image drops joint-state-publisher and tf2-ros, which
  nothing in it runs.
- OvcsMini reads OVCS_SIM in one place and names the VESC's minimum
  ERPM beside the other simulated figures; its README splits the
  obstacle sources and says BackUp runs at the VMS's floor.
- The Nav2 launch file no longer says every VMS floors slow speeds,
  and the bridge firmware's runtime.exs names the two build targets.

Assisted-by: Claude:claude-opus-5-5

File: vehicles/ovcs_mini/description/gazebo_ackermann.xacro (robot description, xacro)
@@ -1,34 +1,13 @@
 <?xml version="1.0"?>
 <!--
-  Ackermann drive for Gazebo Jetty (gz-sim 10).
-  This is the part that could not be carried over from
-  open-vehicle-control-system/traxxas. That model used
-  `libgazebo_ros_ackermann_drive.so`, a **Gazebo Classic** plugin.
-  Classic is end-of-life and the plugin exists in no modern Gazebo;
-  the replacement is Gazebo's own `AckermannSteering` system, reached
-  through `ros_gz_bridge` rather than by linking ROS into the plugin.
-  Every geometry value below is read from the properties in
-  `ovcs_mini.urdf.xacro`, never retyped. That matters because of the
-  failure the previous model shipped with: 0.1 m wheels declared
-  against a real 0.0548.
-  The shape of that failure under gz-sim 10 is the opposite of what
-  one would expect, and was measured rather than assumed. The radius cancels in the
-  plugin — commanded speed is divided by it to get a joint velocity,
-  and the joint velocity is multiplied by it again to get odometry —
-  so `/odom` reads a flawless 1.000 m/s while the car actually crawls
-  at 0.548. The vehicle *reports* correctly and **drives** wrong.
-  Which means `/odom` cannot catch it: compare the physical joint
-  velocity from `/joint_states` against what odometry claims.
-  Tag names here were read out of the shipped
-  `libgz-sim-ackermann-steering-system.so` and the reference world
-  `worlds/ackermann_steering.sdf`, not recalled — and re-checked
-  against gz-sim 10 after the move from Harmonic, where the set turned
-  out to be unchanged. An unrecognised tag is silently ignored and the
-  car simply does not move, so guessing is expensive.
-  Note the absence of a `<topic>` tag: the command topic is left at
-  the system's default, `/model/ovcs_mini/cmd_vel`, and bridged to
-  `/simulator/drive` on the ROS side, where the ROS bridge's simulated
-  hardware publishes it. `<odom_topic>`, `<tf_topic>` and
-  `<child_frame_id>` are set because they are confirmed to exist.
+  Gazebo's AckermannSteering system drives the model; the ROS bridge's
+  simulated hardware commands it on `/simulator/drive`, bridged from the
+  system's default command topic, `/model/ovcs_mini/cmd_vel`, which no
+  tag renames. Every geometry value is read from `ovcs_mini.urdf.xacro`'s
+  properties. The system's own odometry is not bridged: the bridge owns
+  `/odom`, and `OdometryPublisher` gives ground truth on `/simulator/odom`.
+  Tag names come from the shipped
+  `libgz-sim-ackermann-steering-system.so`: an unrecognised tag is
+  ignored without a word.
 -->
 <robot xmlns:xacro="http://www.ros.org/wiki/xacro">
@@ -64,22 +43,8 @@
       <min_acceleration>-10.0</min_acceleration>
       <max_acceleration>10.0</max_acceleration>
-      <odom_topic>/odom</odom_topic>
-      <tf_topic>/tf</tf_topic>
-      <!-- Without this the plugin derives the odometry frame from the
-           model name and publishes `ovcs_mini/odom`, which is not the
-           ROS convention and which Nav2 rejects outright: every costmap
-           logs `Invalid frame ID "odom" ... frame does not exist` and
-           never activates. `frame_id` was read out of the shipped
-           libgz-sim-ackermann-steering-system.so, like the rest of
-           these tags. -->
-      <frame_id>odom</frame_id>
-      <child_frame_id>base_link</child_frame_id>
-      <odom_publish_frequency>50</odom_publish_frequency>
     </plugin>
-    <!-- Ground truth: the model's pose as the physics has it, which the
-         steering system's odometry above is not, it follows the wheels.
-         Its transform goes to a topic nothing bridges: the odom frame
-         belongs to whichever odometry Nav2 navigates by. Tags read out
-         of the shipped libgz-sim-odometry-publisher-system.so. -->
+    <!-- Ground truth: the model's pose as the physics has it. Its
+         transform goes to a topic nothing bridges: the odom frame belongs
+         to the odometry Nav2 navigates by. -->
     <plugin filename="gz-sim-odometry-publisher-system"
             name="gz::sim::systems::OdometryPublisher">
@@ -91,6 +56,6 @@
       <odom_publish_frequency>50</odom_publish_frequency>
     </plugin>
-    <!-- Joint positions, so robot_state_publisher can move the wheels
-         and steering in a viewer rather than showing a rigid model. -->
+    <!-- Joint positions: the simulated hardware measures the wheels from
+         them, and robot_state_publisher moves the wheels in a viewer. -->
     <plugin filename="gz-sim-joint-state-publisher-system"
             name="gz::sim::systems::JointStatePublisher">

File: vehicles/ovcs_mini/description/ovcs_mini.urdf.xacro (robot description, xacro)
@@ -9,5 +9,6 @@
     wheelbase   324 mm
     track       296 mm (centre-to-centre in this model; UNVERIFIED)
-    tyre        109.5 mm diameter -> 54.75 mm radius
+    wheel radius 52.2 mm, as `OvcsMini.geometry/0` (the catalogue's
+                109.5 mm tyre diameter gives 54.75 mm)
     stock envelope 568 x 296 x 193 mm (not the Baja shell)
     mass        2.41 kg (UNVERIFIED with battery and OVCS equipment)
@@ -66,8 +67,13 @@
   <xacro:property name="imu_mass" value="0.005" />
   <xacro:property name="ray_sensor_mass" value="0.005" />
-  <!-- The drive force the simulated hardware gives the VESC's 10 A at its
-       0.5 m/s² per ampere (`OvcsMini`), shared by the four wheels: a
-       wheel held back stalls instead of spinning at the commanded speed. -->
-  <xacro:property name="wheel_max_torque" value="${total_mass * 0.5 * 10 * wheel_radius / 4}" />
+  <!-- As the VMS composer's maximum motor current and the simulated
+       hardware's acceleration per ampere (`OvcsMini`); geometry_test.exs
+       checks both. -->
+  <xacro:property name="max_motor_current" value="10" />
+  <xacro:property name="simulated_acceleration_per_ampere" value="0.5" />
+  <!-- The drive force at the maximum current, shared by the four wheels:
+       a wheel held back stalls instead of spinning at the commanded speed. -->
+  <xacro:property name="wheel_max_torque"
+                  value="${total_mass * simulated_acceleration_per_ampere * max_motor_current * wheel_radius / 4}" />
   <!-- ── Derived ────────────────────────────────────────────────── -->
   <xacro:property name="half_wheelbase" value="${wheelbase / 2}" />
@@ -75,5 +81,5 @@
   <!-- Residual mass after all separately modelled links, including sensors. -->
   <xacro:property name="chassis_mass"
-                  value="${total_mass - 4 * wheel_mass - 2 * steering_mass - 2 * camera_mass - imu_mass}" />
+                  value="${total_mass - 4 * wheel_mass - 2 * steering_mass - 2 * camera_mass - imu_mass - 3 * ray_sensor_mass}" />
   <xacro:property name="tub_z" value="${ground_clearance + tub_height / 2}" />
   <!-- Estimated virtual bicycle steering limit, not the inner-wheel joint limit. -->
@@ -161,7 +167,7 @@
        only orientation is consumed. 100 Hz is the BNO085's cadence. -->
   <xacro:sim_imu name="imu" x="0" y="0" z="0.05" rate="100" />
-  <!-- Mounts as the ROS bridge's static transforms have them
-       (`OvcsMini`'s `lidar_transform/0`, `rear_ultrasound_transforms/0`).
-       The lidar's row stops a step short of +π, which would repeat its first ray. -->
+  <!-- Mounts as the ROS bridge's static transforms have them; geometry_test.exs
+       checks them. The lidar's row stops a step short of +π, which would
+       repeat its first ray. -->
   <xacro:sim_ray name="lidar" x="-0.137" y="0" z="0.205" yaw="0"
                  topic="scan_raw" samples="500"

Commit message: Give the OVCS Mini model a servo-fast steering gain
AckermannSteering drives the steering joints at steer_p_gain radians
per second per radian of error, and its default of 1 is a one-second
servo: while the planner kept adjusting, the joints peaked at 0.42 of
the 0.66 rad lock and the model turned at 0.76 of the 1.77 1/m it was
commanded. At 20 it reaches 1.62.

Assisted-by: Claude:claude-opus-5-5

File: vehicles/ovcs_mini/description/gazebo_ackermann.xacro (robot description, xacro)
@@ -35,4 +35,7 @@
       <kingpin_width>${kingpin_width}</kingpin_width>
       <steering_limit>${gazebo_steering_limit}</steering_limit>
+      <!-- Steering joint speed per radian of error, capped by the joint's
+           velocity limit. -->
+      <steer_p_gain>${steering_servo_gain}</steer_p_gain>
       <!-- ESTIMATE. A stock Slash 4x4 does roughly 30 mph; reverse is
            geared slower. Acceleration limits keep the velocity

File: vehicles/ovcs_mini/description/ovcs_mini.urdf.xacro (robot description, xacro)
@@ -92,4 +92,6 @@
   <!-- Gazebo 10 velocity mode uses L / sin(parameter), not L / tan(parameter). -->
   <xacro:property name="gazebo_steering_limit" value="${asin(tan(steering_limit))}" />
+  <!-- ESTIMATE: an RC servo settles in tens of milliseconds. -->
+  <xacro:property name="steering_servo_gain" value="20.0" />
   <!-- Stereo geometry. -->
   <xacro:property name="baseline" value="0.090" />
