Commit message: Serve the vehicle's meshes to Foxglove
The expanded URDF named its meshes by a file path that existed only
where xacro ran, so Foxglove drew the OVCS Mini without tyres on the
vehicle and in simulation. Foxglove fetches a model's meshes through
foxglove_bridge only as package:// URIs.

Models now name their meshes under a mesh_uri xacro argument, which the
framework sets to package://ovcs_description/meshes. The shared ROS
image registers that package at /opt/ovcs/description, which the local
foxglove_bridge mounts and, on the vehicle, `ovcs compute stage` fills:
the image is built from the compute source root, like Nav2's, with a
vehicle layer on both when the release uses published images. Gazebo
finds the package on GZ_SIM_RESOURCE_PATH. The OVCS Mini's layouts draw
/robot_description in their 3D panels, with Z-up meshes: Foxglove
assumes Y-up and would turn the wheels 90°.

Assisted-by: Claude:claude-opus-5-5

File: vehicles/ovcs_mini/description/ovcs_mini.urdf (robot description, URDF)
Before this commit: robot ovcs_mini, 16 links, 15 joints
Links:
- link front_left_wheel: geometry collision cylinder length=0.045 radius=0.0522; visual mesh filename=package://ovcs_description/meshes/rim.stl scale=0.0522 0.0522 0.045
- link front_right_wheel: geometry collision cylinder length=0.045 radius=0.0522; visual mesh filename=package://ovcs_description/meshes/rim.stl scale=0.0522 0.0522 0.045
- link rear_left_wheel: geometry collision cylinder length=0.045 radius=0.0522; visual mesh filename=package://ovcs_description/meshes/rim.stl scale=0.0522 0.0522 0.045
- link rear_right_wheel: geometry collision cylinder length=0.045 radius=0.0522; visual mesh filename=package://ovcs_description/meshes/rim.stl scale=0.0522 0.0522 0.045

File: vehicles/ovcs_mini/description/visuals.xacro (robot description, xacro)
@@ -1,7 +1,7 @@
 <?xml version="1.0"?>
 <robot xmlns:xacro="http://www.ros.org/wiki/xacro">
-  <xacro:arg name="mesh_dir" default="${xacro.abs_filename('meshes')}" />
+  <xacro:arg name="mesh_uri" default="file://${xacro.abs_filename('meshes')}" />
   <xacro:arg name="show_body" default="false" />
-  <xacro:property name="mesh_dir" value="$(arg mesh_dir)" />
+  <xacro:property name="mesh_uri" value="$(arg mesh_uri)" />
   <material name="shell_blue"><color rgba="0.025 0.24 0.75 1" /></material>
   <material name="window_dark"><color rgba="0.025 0.045 0.065 1" /></material>
@@ -19,5 +19,5 @@
     <visual name="${name}">
       <origin xyz="0 0 ${z}" />
-      <geometry><mesh filename="file://${mesh_dir}/${name}.stl" scale="${scale}" /></geometry>
+      <geometry><mesh filename="${mesh_uri}/${name}.stl" scale="${scale}" /></geometry>
       <material name="${material}" />
     </visual>
