Commit message: Publish the vehicle's URDF with robot_state_publisher
The Nav2 image runs robot_state_publisher from the vehicle's expanded
URDF, which `ovcs compute stage` stages beside the Nav2 parameters. The
car and the simulator now publish the frame tree the same way, every
fixed joint included, so the OVCS Mini's bridges publish no static
transforms. The simulator's launch runs its own, so the simulated nav2
service starts with `robot_state_publisher:=false`.

Assisted-by: Claude:claude-opus-5-5

File: libraries/ovcs_vehicle/test/fixtures/robot.urdf (robot description, URDF)
Before this commit: robot fixture, 7 links, 6 joints
Links:
- removed link camera_link
- removed link camera_optical
- removed link lidar_link
Joints:
- removed joint camera_joint
- removed joint camera_optical_joint
- removed joint lidar_joint

File: vehicles/ovcs_mini/description/ovcs_mini.urdf.xacro (robot description, xacro)
@@ -26,7 +26,7 @@
   bar's height above the ground) read directly off the vehicle.
   ## The expanded URDF
-  `OvcsMini` reads its geometry and the sensor mounts its ROS bridges
-  publish from `ovcs_mini.urdf`, expanded from this file. After an
-  edit, run `mise run urdf`; CI fails while the two differ.
+  `OvcsMini` reads its geometry from `ovcs_mini.urdf`, expanded from
+  this file, and the compute node's robot_state_publisher publishes it.
+  After an edit, run `mise run urdf`; CI fails while the two differ.
 -->
 <robot name="ovcs_mini" xmlns:xacro="http://www.ros.org/wiki/xacro">
